Commit message: Fix macro in simulation urdf

File: black_mouth_control/urdf/simulation.urdf.xacro (robot description, xacro)
@@ -2,9 +2,9 @@
 <robot xmlns:xacro="http://www.ros.org/wiki/xacro" name="quadruped">
     <xacro:macro name="joint_tf">
-        <param name="num">4.99916635e-07 4.99833323e-07</param>
-        <param name="den">1.0 -1.99949913 0.99950012</param>
-        <param name="predict_vel">true</param>
+        <param name="num">1.0</param>
+        <param name="den">1.0</param>
+        <param name="predict_vel">false</param>
     </xacro:macro>
-    <xacro:macro name="leg_joints" params="prefix use_sim">
+    <xacro:macro name="leg_joints" params="prefix">
         <joint name="${prefix}_hip_roll_joint">
             <xacro:joint_tf/>

Commit message: Add controllers config

File: black_mouth_control/urdf/simulation.urdf.xacro (robot description, xacro)
@@ -2,8 +2,9 @@
 <robot xmlns:xacro="http://www.ros.org/wiki/xacro" name="quadruped">
     <xacro:macro name="joint_tf">
-        <param name="num">1.0</param>
-        <param name="den">1.0</param>
-        <!-- <param name="num">0.00213984 0.00214816 0.00420358 0.00477611 0.00609169</param> ARX model -->
-        <!-- <param name="den">1.0 -1.1071699 0.03831938 -0.1805567 0.00378954 0.26499942</param> ARX model -->
+        <!-- <param name="num">1.0</param>
+        <param name="den">1.0</param> -->
+        <!-- ARX model -->
+        <param name="num">0.00213984 0.00214816 0.00420358 0.00477611 0.00609169</param>
+        <param name="den">1.0 -1.1071699 0.03831938 -0.1805567 0.00378954 0.26499942</param>
         <param name="predict_vel">false</param>
     </xacro:macro>
@@ -15,11 +16,5 @@
                 <param name="max">0.52</param>
             </command_interface>
-            <command_interface name="velocity">
-                <!--TODO Review-->>
-                <param name="min">-30</param>
-                <param name="max">30</param>
-            </command_interface>
             <state_interface name="position"/>
-            <state_interface name="velocity"/>
         </joint>
         <joint name="${prefix}_hip_pitch_joint">
@@ -29,11 +24,5 @@
                 <param name="max">0.79</param>
             </command_interface>
-            <command_interface name="velocity">
-                <!--TODO Review-->>
-                <param name="min">-30</param>
-                <param name="max">30</param>
-            </command_interface>
             <state_interface name="position"/>
-            <state_interface name="velocity"/>
         </joint>
         <joint name="${prefix}_elbow_joint">
@@ -43,11 +32,5 @@
                 <param name="max">0.63</param>
             </command_interface>
-            <command_interface name="velocity">
-                <!--TODO Review-->>
-                <param name="min">-30</param>
-                <param name="max">30</param>
-            </command_interface>
             <state_interface name="position"/>
-            <state_interface name="velocity"/>
         </joint>
     </xacro:macro>

File: black_mouth_description/urdf/black_mouth.urdf.xacro (robot description, xacro)
@@ -13,4 +13,5 @@
     <xacro:property name="leg_y_offset" value="0.07"/>
     <xacro:property name="leg_z_offset" value="0.020822"/>
+    <xacro:property name="effort_limit" value="0.01"/>
     <xacro:macro name="leg" params="prefix left front *joint_pose">
         <link name="${prefix}_hip">
@@ -68,6 +69,7 @@
             <child link="${prefix}_hip"/>
             <axis xyz="1 0 0"/>
-            <limit lower="${-M_PI/6}" upper="${M_PI/6}" velocity="5.75" effort="2.5"/>
+            <limit lower="${-M_PI/6}" upper="${M_PI/6}" velocity="5.75" effort="${effort_limit}"/>
             <xacro:insert_block name="joint_pose"/>
+            <!-- <dynamics damping="5.0" friction="5.0" /> -->
         </joint>
         <link name="${prefix}_link_femur">
@@ -122,5 +124,6 @@
             <child link="${prefix}_link_femur"/>
             <axis xyz="0 1 0"/>
-            <limit lower="${-M_PI/4}" upper="${M_PI/4}" velocity="5.75" effort="2.5"/>
+            <limit lower="${-M_PI/4}" upper="${M_PI/4}" velocity="5.75" effort="${effort_limit}"/>
+            <!-- <dynamics damping="5.0" friction="5.0" /> -->
         </joint>
         <link name="${prefix}_tibia">
@@ -144,6 +147,9 @@
         </link>
         <gazebo reference="${prefix}_tibia">
-            <mu1>0.8</mu1>
-            <mu2>0.8</mu2>
+            <mu1>1.0</mu1>
+            <mu2>1.0</mu2>
+            <minDepth>0.0002</minDepth>
+            <kp value="1000000.0"/>
+            <kd value="100.0"/>
             <selfCollide>true</selfCollide>
         </gazebo>
@@ -158,8 +164,10 @@
             <child link="${prefix}_tibia"/>
             <axis xyz="0 1 0"/>
-            <limit lower="${-M_PI/5}" upper="${M_PI/5}" velocity="5.75" effort="2.5"/>
+            <limit lower="${-M_PI/5}" upper="${M_PI/5}" velocity="5.75" effort="${effort_limit}"/>
+            <!-- <dynamics damping="5.0" friction="5.0" /> -->
         </joint>
     </xacro:macro>
-    <link name="base_footprint"/>
+    <link name="base_footprint">
+    </link>
     <link name="base_link">
         <visual>
@@ -203,5 +211,5 @@
         <origin xyz="${-leg_x_offset} ${leg_y_offset} ${leg_z_offset}" rpy="0.0 0.0 0.0"/>
     </xacro:leg>
-    <xacro:leg prefix="back_right" left="${False}" front="${False}" >
+    <xacro:leg prefix="back_right" left="${False}" front="${False}">
         <origin xyz="${-leg_x_offset} ${-leg_y_offset} ${leg_z_offset}" rpy="0.0 0.0 0.0"/>
     </xacro:leg>
@@ -216,20 +224,22 @@
         <gravity>true</gravity>
         <sensor name="imu_sensor" type="imu">
-        <always_on>true</always_on>
-        <update_rate>100</update_rate>
-        <visualize>true</visualize>
-        <topic>__default_topic__</topic>
-        <plugin filename="libgazebo_ros_imu_sensor.so" name="imu_plugin">
-            <topicName>imu</topicName>
-            <bodyName>imu_link</bodyName>
-            <updateRateHZ>10.0</updateRateHZ>
-            <gaussianNoise>0.0</gaussianNoise>
-            <xyzOffset>0 0 0</xyzOffset>
-            <rpyOffset>0 0 0</rpyOffset>
-            <frameName>imu_link</frameName>
-            <initialOrientationAsReference>false</initialOrientationAsReference>
-        </plugin>
-        <pose>0 0 0 0 0 0</pose>
+            <always_on>true</always_on>
+            <update_rate>100</update_rate>
+            <visualize>true</visualize>
+            <topic>__default_topic__</topic>
+            <plugin filename="libgazebo_ros_imu_sensor.so" name="imu_plugin">
+                <topicName>imu</topicName>
+                <bodyName>imu_link</bodyName>
+                <updateRateHZ>10.0</updateRateHZ>
+                <gaussianNoise>0.0</gaussianNoise>
+                <xyzOffset>0 0 0</xyzOffset>
+                <rpyOffset>0 0 0</rpyOffset>
+                <frameName>imu_link</frameName>
+                <initialOrientationAsReference>false</initialOrientationAsReference>
+            </plugin>
+            <pose>0 0 0 0 0 0</pose>
         </sensor>
     </gazebo>
+    <!-- Ros2 Control -->
+    <xacro:include filename="$(find black_mouth_control)/urdf/simulation.urdf.xacro"/>
 </robot>
