Commit message: update urdf

File: black_mouth_description/urdf/black_mouth.urdf.xacro (robot description, xacro)
@@ -23,17 +23,21 @@
         <link name="${prefix}_femur">
             <visual>
-                <origin xyz="0.0 0.0 ${-femur_length/2} " rpy="${M_PI/2} 0.0  0.0"/>
-                <geometry>
-                    <box size="0.035 ${femur_length} 0.036"/>
-                </geometry>
-                <!-- <mesh filename="file://$(find black_mouth_description)/meshes/left_femur.dae" /> -->
-                <material name="Green">
-                    <color rgba="0.0 1.0 0.0 1.0"/>
-                </material>
+                <xacro:if value="${left}">
+                    <origin xyz="0.0 -0.006 0.0" rpy="${M_PI/2} 0.0 ${-M_PI/2} "/>
+                    <geometry>
+                        <mesh filename="file://$(find black_mouth_description)/meshes/left_femur.dae" />
+                    </geometry>
+                </xacro:if>
+                <xacro:unless value="${left}">
+                    <origin xyz="0.0 0.006 0.0" rpy="${M_PI/2} 0.0 ${-M_PI/2} "/>
+                    <geometry>
+                        <mesh filename="file://$(find black_mouth_description)/meshes/right_femur.dae" />
+                    </geometry>
+                </xacro:unless>
             </visual>
             <collision>
-                <origin xyz="0.0 0.0 ${-femur_length/2} " rpy="${M_PI/2} 0.0  0.0"/>
+                <origin xyz="0.0 0.0 ${-femur_length/3}" rpy="${M_PI/2} 0.0 ${-M_PI/2} "/>
                 <geometry>
-                    <box size="0.035 ${femur_length} 0.036"/>
+                    <box size="0.035 ${femur_length} 0.036" />
                 </geometry>
             </collision>
@@ -41,5 +45,5 @@
                 <mass value="1.0"/>
                 <origin xyz="0.0 0.0 0.0" rpy="0.0 0.0 0.0"/>
-                <inertia ixx="1e-6" ixy="0.0" ixz="0.0" iyy="1e-6" iyz="0.0" izz="1e-6"/>
+                <inertia ixx="4.182" ixy="-0.002532" ixz="-0.011148" iyy="8.258" iyz="0.001" izz="11.706"/>
             </inertial>
         </link>
@@ -50,8 +54,8 @@
             <limit lower="-3.14159" upper="3.14159" velocity="50.0" effort="1000.0"/>
             <xacro:if value="${left}">
-                <origin xyz="0 0.045 0.0" rpy="0.0 0.0 0.0"/>
+                <origin xyz="0 0.05 0.0" rpy="0.0 0.0 0.0"/>
             </xacro:if>
             <xacro:unless value="${left}">
-                <origin xyz="0 -0.045 0.0" rpy="0.0 0.0 0.0"/>
+                <origin xyz="0 -0.05 0.0" rpy="0.0 0.0 0.0"/>
             </xacro:unless>
         </joint>
@@ -59,17 +63,14 @@
             <visual>
             <xacro:if value="${left}">
-                <!-- <origin xyz="0 0.045 0.0" rpy="0.0 0.0 0.0"/>
-                <mesh filename="file://$(find black_mouth_description)/meshes/left_tibia.dae" /> -->
-                <origin xyz="0.0 0.0 ${-tibia_length/2} " rpy="${M_PI/2} 0.0  0.0"/>
+                <origin xyz="0.0 0.0 0.0 " rpy="0.0 0.0 0.0"/>
                 <geometry>
-                    <box size="0.035 ${tibia_length} 0.036"/>
+                    <mesh filename="file://$(find black_mouth_description)/meshes/left_tibia.dae" />
                 </geometry>
-                <material name="Red">
-                    <color rgba="1.0 .0 0.0 1.0"/>
-                </material>
             </xacro:if>
             <xacro:unless value="${left}">
-                <origin xyz="0 -0.045 0.0" rpy="0.0 0.0 0.0"/>
-                <mesh filename="file://$(find black_mouth_description)/meshes/right_tibia.dae" />
+                <origin xyz="0.0 0.0 0.0 " rpy="0.0 0.0 0.0"/>
+                <geometry>
+                    <mesh filename="file://$(find black_mouth_description)/meshes/right_tibia.dae" />
+                </geometry>
             </xacro:unless>
             </visual>
@@ -91,5 +92,5 @@
             <axis xyz="0 1 0"/>
             <limit lower="-3.14159" upper="3.14159" velocity="50.0" effort="1000.0"/>
-            <origin xyz="0.0 0.0 -${femur_length}" rpy="0.0 0.0 0.0"/>
+            <origin xyz="-0.00 0.0 ${-femur_length +0.035}" rpy="0.0 0.0 0.0"/>
         </joint>
     </xacro:macro>
@@ -102,4 +103,5 @@
         </visual>
         <collision>
+            <origin xyz="0.0 0.0 ${body_height/2}" rpy="0.0 0.0 0.0"/>
             <geometry>
                 <box size="${body_length} ${body_width} ${body_height}" />
@@ -115,5 +117,5 @@
         <parent link="base_footprint"/>
         <child link="base_link"/>
-        <origin xyz="0.0 0.0 0.15" rpy="0.0 0.0 0.0"/>
+        <origin xyz="0.0 0.0 0.15" rpy="0.0 0.0 ${M_PI/2}"/>
     </joint>
     <xacro:leg prefix="front_left" left="${True}" >
@@ -129,3 +131,30 @@
         <origin xyz="-0.11 -0.07 0.020822" rpy="0.0 0.0 0.0"/>
     </xacro:leg>
+    <link name="imu_link"/>
+    <joint name="imu_joint" type="fixed">
+        <origin xyz="0.0 0.0 0.0" rpy="0.0 0.0 0.0"/>
+        <parent link="base_link"/>
+        <child link="imu_link"/>
+        <axis xyz="0.075 0.0 0.0738"/>
+    </joint>
+    <gazebo reference="imu_link">
+    <gravity>true</gravity>
+    <sensor name="imu_sensor" type="imu">
+      <always_on>true</always_on>
+      <update_rate>100</update_rate>
+      <visualize>true</visualize>
+      <topic>__default_topic__</topic>
+      <plugin filename="libgazebo_ros_imu_sensor.so" name="imu_plugin">
+        <topicName>imu</topicName>
+        <bodyName>imu_link</bodyName>
+        <updateRateHZ>10.0</updateRateHZ>
+        <gaussianNoise>0.0</gaussianNoise>
+        <xyzOffset>0 0 0</xyzOffset>
+        <rpyOffset>0 0 0</rpyOffset>
+        <frameName>imu_link</frameName>
+        <initialOrientationAsReference>false</initialOrientationAsReference>
+      </plugin>
+      <pose>0 0 0 0 0 0</pose>
+    </sensor>
+  </gazebo>
 </robot>

Commit message: update urdf

File: black_mouth_description/urdf/black_mouth.urdf.xacro (robot description, xacro)
@@ -3,5 +3,5 @@
     <xacro:property name="M_PI" value="3.1415"/>
     <xacro:property name="body_length" value="0.262"/>
-    <xacro:property name="body_width" value="0.162"/>
+    <xacro:property name="body_width" value="0.11"/>
     <xacro:property name="body_height" value="0.062"/>
     <xacro:property name="hip_length" value="0.1"/>
@@ -12,6 +12,34 @@
     <xacro:property name="leg_y_offset" value="${body_width/2 + hip_length/2}"/>
     <xacro:property name="leg_z_offset" value="${-body_height/4}"/>
-    <xacro:macro name="leg" params="prefix left *joint_pose ">
-        <link name="${prefix}_hip"/>
+    <xacro:macro name="leg" params="prefix left front *joint_pose ">
+        <link name="${prefix}_hip">
+            <inertial>
+                <origin xyz="0.0 0.0 0.0" rpy="0.0 0.0 0.0"/>
+                <mass value="0.7"/>
+                <inertia ixx="13.0" ixy="0.689" ixz="0.02" iyy="18.242" iyz="0.008" izz="22.035"/>
+            </inertial>
+            <visual>
+                <xacro:if value="${front}">
+                    <origin xyz="0.0 0.0 0.0" rpy="0.0 ${-M_PI/2} ${-M_PI/2}"/>
+                </xacro:if>
+                <xacro:unless value="${front}">
+                    <origin xyz="0.0 0.0 0.0" rpy="0.0 ${M_PI/2} ${M_PI/2}"/>
+                </xacro:unless>
+                <geometry>
+                        <mesh filename="file://$(find black_mouth_description)/meshes/dynamixel.dae" />
+                </geometry>
+            </visual>
+            <collision>
+                <xacro:if value="${front}">
+                    <origin xyz="-0.015 0.0 0.0" rpy="0.0 0.0 0.0"/>
+                </xacro:if>
+                <xacro:unless value="${front}">
+                    <origin xyz="0.015 0.0 0.0" rpy="0.0 0.0 0.0"/>
+                </xacro:unless>
+                <geometry>
+                    <box size="0.05 0.03 0.035"/>
+                </geometry>
+            </collision>
+        </link>
         <joint name="${prefix}_hip_roll_joint" type="revolute">
             <parent link="base_link"/>
@@ -99,5 +127,5 @@
         <visual>
             <geometry>
-                <mesh filename="file://$(find black_mouth_description)/meshes/Chassis_assembly.dae" />
+                <mesh filename="file://$(find black_mouth_description)/meshes/base_link.dae" />
             </geometry>
         </visual>
@@ -105,5 +133,5 @@
             <origin xyz="0.0 0.0 ${body_height/2}" rpy="0.0 0.0 0.0"/>
             <geometry>
-                <box size="${body_length} ${body_width} ${body_height}" />
+                <box size="${body_length} ${body_width-0.001} ${body_height}" />
             </geometry>
         </collision>
@@ -119,15 +147,15 @@
         <origin xyz="0.0 0.0 0.15" rpy="0.0 0.0 ${M_PI/2}"/>
     </joint>
-    <xacro:leg prefix="front_left" left="${True}" >
-        <origin xyz="0.11 0.07 0.020822" rpy="0.0 0.0 0.0"/>
+    <xacro:leg prefix="front_left" left="${True}" front="${True}">
+        <origin xyz="${body_length/2 -0.02} 0.07 0.020822" rpy="0.0 0.0 0.0"/>
     </xacro:leg>
-    <xacro:leg prefix="front_right" left="${False}">
-        <origin xyz="0.11 -0.07 0.020822" rpy="0.0 0.0 0.0"/>
+    <xacro:leg prefix="front_right" left="${False}" front="${True}">
+        <origin xyz="${body_length/2 -0.02} -0.07 0.020822" rpy="0.0 0.0 0.0"/>
     </xacro:leg>
-    <xacro:leg prefix="back_left" left="${True}">
-        <origin xyz="-0.11 0.07 0.020822" rpy="0.0 0.0 0.0"/>
+    <xacro:leg prefix="back_left" left="${True}" front="${False}">
+        <origin xyz="${-(body_length/2 -0.02)} 0.07 0.020822" rpy="0.0 0.0 0.0"/>
     </xacro:leg>
-    <xacro:leg prefix="back_right" left="${False}" >
-        <origin xyz="-0.11 -0.07 0.020822" rpy="0.0 0.0 0.0"/>
+    <xacro:leg prefix="back_right" left="${False}" front="${False}" >
+        <origin xyz="${-(body_length/2 -0.02)} -0.07 0.020822" rpy="0.0 0.0 0.0"/>
     </xacro:leg>
     <link name="imu_link"/>

Commit message: update urdf

File: black_mouth_description/urdf/black_mouth.urdf.xacro (robot description, xacro)
@@ -49,23 +49,23 @@
             <xacro:insert_block name="joint_pose"/>
         </joint>
-        <link name="${prefix}_femur">
+        <link name="${prefix}_motor_femur">
             <visual>
                 <xacro:if value="${left}">
-                    <origin xyz="0.0 -0.006 0.0" rpy="${M_PI/2} 0.0 ${-M_PI/2} "/>
-                    <geometry>
-                        <mesh filename="file://$(find black_mouth_description)/meshes/left_femur.dae" />
+                    <origin xyz="0.0 -0.001 0.0" rpy="${M_PI/2} 0.0 ${-M_PI/2} "/>
+                    <geometry>
+                        <mesh filename="file://$(find black_mouth_description)/meshes/dynamixel.dae" />
                     </geometry>
                 </xacro:if>
                 <xacro:unless value="${left}">
-                    <origin xyz="0.0 0.006 0.0" rpy="${M_PI/2} 0.0 ${-M_PI/2} "/>
-                    <geometry>
-                        <mesh filename="file://$(find black_mouth_description)/meshes/right_femur.dae" />
-                    </geometry>
-                </xacro:unless>
-            </visual>
-            <collision>
-                <origin xyz="0.0 0.0 ${-femur_length/3}" rpy="${M_PI/2} 0.0 ${-M_PI/2} "/>
-                <geometry>
-                    <box size="0.035 ${femur_length} 0.036" />
+                    <origin xyz="0.0 0.001 0.0" rpy="${M_PI/2} 0.0 ${-M_PI/2} "/>
+                    <geometry>
+                        <mesh filename="file://$(find black_mouth_description)/meshes/dynamixel.dae"/>
+                    </geometry>
+                </xacro:unless>
+            </visual>
+            <collision>
+                <origin xyz="0.0 0.0 -0.015" rpy="0.0 ${-M_PI/2} 0.0 "/>
+                <geometry>
+                    <box size="0.05 0.03 0.035"/>
                 </geometry>
             </collision>
@@ -78,18 +78,50 @@
         <joint name="${prefix}_hip_pitch_joint" type="revolute">
             <parent link="${prefix}_hip"/>
-            <child link="${prefix}_femur"/>
+            <child link="${prefix}_motor_femur"/>
             <axis xyz="0 1 0"/>
             <limit lower="-3.14159" upper="3.14159" velocity="50.0" effort="1000.0"/>
             <xacro:if value="${left}">
-                <origin xyz="0 0.05 0.0" rpy="0.0 0.0 0.0"/>
+                <origin xyz="0 0.04 0.0" rpy="0.0 0.0 0.0"/>
             </xacro:if>
             <xacro:unless value="${left}">
-                <origin xyz="0 -0.05 0.0" rpy="0.0 0.0 0.0"/>
+                <origin xyz="0 -0.04 0.0" rpy="0.0 0.0 0.0"/>
             </xacro:unless>
         </joint>
+        <link name="${prefix}_link_femur">
+            <visual>
+                <xacro:if value="${left}">
+                    <origin xyz="0.0 0 0.035" rpy="${M_PI/2} 0.0 ${-M_PI/2} "/>
+                    <geometry>
+                        <mesh filename="file://$(find black_mouth_description)/meshes/left_femur.dae" />
+                    </geometry>
+                </xacro:if>
+                <xacro:unless value="${left}">
+                    <origin xyz="0.0 0.0 0.035" rpy="${M_PI/2} 0.0 ${-M_PI/2} "/>
+                    <geometry>
+                        <mesh filename="file://$(find black_mouth_description)/meshes/right_femur.dae" />
+                    </geometry>
+                </xacro:unless>
+            </visual>
+            <collision>
+                <origin xyz="0.0 0.0 -0.04" rpy="${M_PI/2} 0.0 ${-M_PI/2} "/>
+                <geometry>
+                    <box size="0.035 ${femur_length*2/3} 0.036" />
+                </geometry>
+            </collision>
+            <inertial>
+                <mass value="1.0"/>
+                <origin xyz="0.0 0.0 0.0" rpy="0.0 0.0 0.0"/>
+                <inertia ixx="4.182" ixy="-0.002532" ixz="-0.011148" iyy="8.258" iyz="0.001" izz="11.706"/>
+            </inertial>
+        </link>
+        <joint name="${prefix}_femur_joint" type="fixed">
+            <parent link="${prefix}_motor_femur"/>
+            <child link="${prefix}_link_femur"/>
+            <origin xyz="0.00 0.0 -0.05" rpy="0.0 0.0 0.0"/>
+        </joint>
         <link name="${prefix}_tibia">
             <visual>
             <xacro:if value="${left}">
-                <origin xyz="0.0 0.0 0.0 " rpy="0.0 0.0 0.0"/>
+                <origin xyz="0.0 0.007 0.0 " rpy="0.0 0.0 0.0"/>
                 <geometry>
                     <mesh filename="file://$(find black_mouth_description)/meshes/left_tibia.dae" />
@@ -97,5 +129,5 @@
             </xacro:if>
             <xacro:unless value="${left}">
-                <origin xyz="0.0 0.0 0.0 " rpy="0.0 0.0 0.0"/>
+                <origin xyz="0.0 -0.007 0.0 " rpy="0.0 0.0 0.0"/>
                 <geometry>
                     <mesh filename="file://$(find black_mouth_description)/meshes/right_tibia.dae" />
@@ -104,7 +136,7 @@
             </visual>
             <collision>
-                <origin xyz="0.0 0.0 ${-tibia_length/2} " rpy="${M_PI/2} 0.0  0.0"/>
-                <geometry>
-                    <box size="0.035 ${tibia_length} 0.036"/>
+                <origin xyz="0.0 0.0 ${-tibia_length/2 -0.0025} " rpy="${M_PI/2} 0.0  0.0"/>
+                <geometry>
+                    <box size="0.035 ${tibia_length -0.02} 0.036"/>
                 </geometry>
             </collision>
@@ -116,9 +148,9 @@
         </link>
         <joint name="${prefix}_elbow_joint" type="revolute">
-            <parent link="${prefix}_femur"/>
+            <parent link="${prefix}_link_femur"/>
             <child link="${prefix}_tibia"/>
             <axis xyz="0 1 0"/>
             <limit lower="-3.14159" upper="3.14159" velocity="50.0" effort="1000.0"/>
-            <origin xyz="-0.00 0.0 ${-femur_length +0.035}" rpy="0.0 0.0 0.0"/>
+            <origin xyz="-0.00 0.0 ${-femur_length +0.065}" rpy="0.0 0.0 0.0"/>
         </joint>
     </xacro:macro>
@@ -145,5 +177,5 @@
         <parent link="base_footprint"/>
         <child link="base_link"/>
-        <origin xyz="0.0 0.0 0.15" rpy="0.0 0.0 ${M_PI/2}"/>
+        <origin xyz="0.0 0.0 0.15" rpy="0.0 0.0 0.0"/>
     </joint>
     <xacro:leg prefix="front_left" left="${True}" front="${True}">
