Commit message: Add foot and hip_fixed links to URDF and compute IK in ros service

File: black_mouth_description/urdf/black_mouth.urdf.xacro (robot description, xacro)
@@ -14,4 +14,20 @@
     <xacro:property name="leg_z_offset" value="0.020822"/>
     <xacro:macro name="leg" params="prefix left front *joint_pose">
+        <link name="${prefix}_hip_fixed">
+            <collision>
+                <geometry>
+                    <sphere radius="0.001"/>
+                </geometry>
+            </collision>
+            <inertial>
+                <mass value="0.001"/>
+                <inertia ixx="1e-6" ixy="0.0" ixz="0.0" iyy="1e-6" iyz="0.0" izz="1e-6"/>
+            </inertial>
+        </link>
+        <joint name="${prefix}_hip_fixed_joint" type="fixed">
+            <parent link="base_link"/>
+            <child link="${prefix}_hip_fixed"/>
+            <xacro:insert_block name="joint_pose"/>
+        </joint>
         <link name="${prefix}_hip">
             <xacro:if value="${front}">
@@ -65,11 +81,12 @@
         </gazebo>
         <joint name="${prefix}_hip_roll_joint" type="revolute">
-            <parent link="base_link"/>
+            <origin xyz="0.0 0.0 0.0" rpy="0.0 0.0 0.0"/>
+            <parent link="${prefix}_hip_fixed"/>
             <child link="${prefix}_hip"/>
             <axis xyz="1 0 0"/>
-            <limit lower="${-M_PI/6}" upper="${M_PI/6}" velocity="5.75" effort="2.5"/>
-            <xacro:insert_block name="joint_pose"/>
-        </joint>
-        <link name="${prefix}_link_femur">
+            <!-- <limit lower="${-M_PI/6}" upper="${M_PI/6}" velocity="5.75" effort="2.5"/> -->
+            <limit lower="${-M_PI}" upper="${M_PI}" velocity="5.75" effort="2.5"/>
+        </joint>
+        <link name="${prefix}_femur">
             <visual>
                 <origin xyz="0.0 0 ${-femur_offset}" rpy="0.0 0.0 0.0 "/>
@@ -107,5 +124,5 @@
             </inertial>
         </link>
-        <gazebo reference="${prefix}_link_femur">
+        <gazebo reference="${prefix}_femur">
             <mu1>0.4</mu1>
             <mu2>0.4</mu2>
@@ -114,13 +131,16 @@
         <joint name="${prefix}_hip_pitch_joint" type="revolute">
             <xacro:if value="${left}">
-                <origin xyz="0 ${hip_length} 0.0" rpy="0.0 ${M_PI/4} 0.0"/>
+                <!-- <origin xyz="0 ${hip_length} 0.0" rpy="0.0 ${M_PI/4} 0.0"/> -->
+                <origin xyz="0 ${hip_length} 0.0" rpy="0.0 0.0 0.0"/>
             </xacro:if>
             <xacro:unless value="${left}">
-                <origin xyz="0 ${-hip_length} 0.0" rpy="0.0 ${M_PI/4} 0.0"/>
+                <!-- <origin xyz="0 ${-hip_length} 0.0" rpy="0.0 ${M_PI/4} 0.0"/> -->
+                <origin xyz="0 ${-hip_length} 0.0" rpy="0.0 0.0 0.0"/>
             </xacro:unless>
             <parent link="${prefix}_hip"/>
-            <child link="${prefix}_link_femur"/>
+            <child link="${prefix}_femur"/>
             <axis xyz="0 1 0"/>
-            <limit lower="${-M_PI/4}" upper="${M_PI/4}" velocity="5.75" effort="2.5"/>
+            <!-- <limit lower="${-M_PI/4}" upper="${M_PI/4}" velocity="5.75" effort="2.5"/> -->
+            <limit lower="${-M_PI}" upper="${M_PI}" velocity="5.75" effort="2.5"/>
         </joint>
         <link name="${prefix}_tibia">
@@ -150,13 +170,22 @@
         <joint name="${prefix}_elbow_joint" type="revolute">
             <xacro:if value="${left}">
-                <origin xyz="0.00 ${femur_thickness/2 - 0.0042} ${-femur_length}" rpy="0.0 ${-M_PI/2} 0.0"/>
+                <!-- <origin xyz="0.00 ${femur_thickness/2 - 0.0042} ${-femur_length}" rpy="0.0 ${-M_PI/2} 0.0"/> -->
+                <origin xyz="0.00 ${femur_thickness/2 - 0.0042} ${-femur_length}" rpy="0.0 0.0 0.0"/>
             </xacro:if>
             <xacro:unless value="${left}">
-                <origin xyz="0.00 ${-femur_thickness/2 + 0.0042} ${-femur_length}" rpy="0.0 ${-M_PI/2} 0.0"/>
+                <!-- <origin xyz="0.00 ${-femur_thickness/2 + 0.0042} ${-femur_length}" rpy="0.0 ${-M_PI/2} 0.0"/> -->
+                <origin xyz="0.00 ${-femur_thickness/2 + 0.0042} ${-femur_length}" rpy="0.0 0.0 0.0"/>
             </xacro:unless>
-            <parent link="${prefix}_link_femur"/>
+            <parent link="${prefix}_femur"/>
             <child link="${prefix}_tibia"/>
             <axis xyz="0 1 0"/>
-            <limit lower="${-M_PI/5}" upper="${M_PI/5}" velocity="5.75" effort="2.5"/>
+            <!-- <limit lower="${-M_PI/5}" upper="${M_PI/5}" velocity="5.75" effort="2.5"/> -->
+            <limit lower="${-M_PI}" upper="${M_PI}" velocity="5.75" effort="2.5"/>
+        </joint>
+        <link name="${prefix}_foot"/>
+        <joint name="${prefix}_foot_joint" type="fixed">
+            <parent link="${prefix}_tibia"/>
+            <child link="${prefix}_foot"/>
+            <origin xyz="0.0 0.0 ${-tibia_length}" rpy="0.0 ${M_PI/4} 0.0"/>
         </joint>
     </xacro:macro>

Commit message: Add foot and hip_fixed links to URDF and compute IK in ros service

File: black_mouth_description/urdf/black_mouth.urdf.xacro (robot description, xacro)
@@ -15,4 +15,20 @@
     <xacro:property name="effort_limit" value="0.01"/>
     <xacro:macro name="leg" params="prefix left front *joint_pose">
+        <link name="${prefix}_hip_fixed">
+            <collision>
+                <geometry>
+                    <sphere radius="0.001"/>
+                </geometry>
+            </collision>
+            <inertial>
+                <mass value="0.001"/>
+                <inertia ixx="1e-6" ixy="0.0" ixz="0.0" iyy="1e-6" iyz="0.0" izz="1e-6"/>
+            </inertial>
+        </link>
+        <joint name="${prefix}_hip_fixed_joint" type="fixed">
+            <parent link="base_link"/>
+            <child link="${prefix}_hip_fixed"/>
+            <xacro:insert_block name="joint_pose"/>
+        </joint>
         <link name="${prefix}_hip">
             <xacro:if value="${front}">
@@ -66,12 +82,12 @@
         </gazebo>
         <joint name="${prefix}_hip_roll_joint" type="revolute">
-            <parent link="base_link"/>
+            <origin xyz="0.0 0.0 0.0" rpy="0.0 0.0 0.0"/>
+            <parent link="${prefix}_hip_fixed"/>
             <child link="${prefix}_hip"/>
             <axis xyz="1 0 0"/>
             <limit lower="${-M_PI/6}" upper="${M_PI/6}" velocity="5.75" effort="${effort_limit}"/>
-            <xacro:insert_block name="joint_pose"/>
             <!-- <dynamics damping="5.0" friction="5.0" /> -->
         </joint>
-        <link name="${prefix}_link_femur">
+        <link name="${prefix}_femur">
             <visual>
                 <origin xyz="0.0 0 ${-femur_offset}" rpy="0.0 0.0 0.0 "/>
@@ -109,5 +125,5 @@
             </inertial>
         </link>
-        <gazebo reference="${prefix}_link_femur">
+        <gazebo reference="${prefix}_femur">
             <mu1>0.4</mu1>
             <mu2>0.4</mu2>
@@ -116,5 +132,6 @@
         <joint name="${prefix}_hip_pitch_joint" type="revolute">
             <xacro:if value="${left}">
-                <origin xyz="0 ${hip_length} 0.0" rpy="0.0 ${M_PI/4} 0.0"/>
+                <!-- <origin xyz="0 ${hip_length} 0.0" rpy="0.0 ${M_PI/4} 0.0"/> -->
+                <origin xyz="0 ${hip_length} 0.0" rpy="0.0 0.0 0.0"/>
             </xacro:if>
             <xacro:unless value="${left}">
@@ -122,5 +139,5 @@
             </xacro:unless>
             <parent link="${prefix}_hip"/>
-            <child link="${prefix}_link_femur"/>
+            <child link="${prefix}_femur"/>
             <axis xyz="0 1 0"/>
             <limit lower="${-M_PI/4}" upper="${M_PI/4}" velocity="5.75" effort="${effort_limit}"/>
@@ -161,9 +178,15 @@
                 <origin xyz="0.00 ${-femur_thickness/2 + 0.0042} ${-femur_length}" rpy="0.0 ${-M_PI/2} 0.0"/>
             </xacro:unless>
-            <parent link="${prefix}_link_femur"/>
+            <parent link="${prefix}_femur"/>
             <child link="${prefix}_tibia"/>
             <axis xyz="0 1 0"/>
             <limit lower="${-M_PI/5}" upper="${M_PI/5}" velocity="5.75" effort="${effort_limit}"/>
             <!-- <dynamics damping="5.0" friction="5.0" /> -->
+        </joint>
+        <link name="${prefix}_foot"/>
+        <joint name="${prefix}_foot_joint" type="fixed">
+            <parent link="${prefix}_tibia"/>
+            <child link="${prefix}_foot"/>
+            <origin xyz="0.0 0.0 ${-tibia_length}" rpy="0.0 ${M_PI/4} 0.0"/>
         </joint>
     </xacro:macro>

Commit message: Add offset to IK and body translation

File: black_mouth_description/urdf/black_mouth.urdf.xacro (robot description, xacro)
@@ -132,6 +132,5 @@
         <joint name="${prefix}_hip_pitch_joint" type="revolute">
             <xacro:if value="${left}">
-                <!-- <origin xyz="0 ${hip_length} 0.0" rpy="0.0 ${M_PI/4} 0.0"/> -->
-                <origin xyz="0 ${hip_length} 0.0" rpy="0.0 0.0 0.0"/>
+                <origin xyz="0 ${hip_length} 0.0" rpy="0.0 ${M_PI/4} 0.0"/>
             </xacro:if>
             <xacro:unless value="${left}">

Commit message: Add offset to IK and body translation

File: black_mouth_description/urdf/black_mouth.urdf.xacro (robot description, xacro)
@@ -85,6 +85,5 @@
             <child link="${prefix}_hip"/>
             <axis xyz="1 0 0"/>
-            <!-- <limit lower="${-M_PI/6}" upper="${M_PI/6}" velocity="5.75" effort="2.5"/> -->
-            <limit lower="${-M_PI}" upper="${M_PI}" velocity="5.75" effort="2.5"/>
+            <limit lower="${-M_PI/6}" upper="${M_PI/6}" velocity="5.75" effort="2.5"/>
         </joint>
         <link name="${prefix}_femur">
@@ -131,16 +130,13 @@
         <joint name="${prefix}_hip_pitch_joint" type="revolute">
             <xacro:if value="${left}">
-                <!-- <origin xyz="0 ${hip_length} 0.0" rpy="0.0 ${M_PI/4} 0.0"/> -->
-                <origin xyz="0 ${hip_length} 0.0" rpy="0.0 0.0 0.0"/>
+                <origin xyz="0 ${hip_length} 0.0" rpy="0.0 ${M_PI/4} 0.0"/>
             </xacro:if>
             <xacro:unless value="${left}">
-                <!-- <origin xyz="0 ${-hip_length} 0.0" rpy="0.0 ${M_PI/4} 0.0"/> -->
-                <origin xyz="0 ${-hip_length} 0.0" rpy="0.0 0.0 0.0"/>
+                <origin xyz="0 ${-hip_length} 0.0" rpy="0.0 ${M_PI/4} 0.0"/>
             </xacro:unless>
             <parent link="${prefix}_hip"/>
             <child link="${prefix}_femur"/>
             <axis xyz="0 1 0"/>
-            <!-- <limit lower="${-M_PI/4}" upper="${M_PI/4}" velocity="5.75" effort="2.5"/> -->
-            <limit lower="${-M_PI}" upper="${M_PI}" velocity="5.75" effort="2.5"/>
+            <limit lower="${-M_PI/4}" upper="${M_PI/4}" velocity="5.75" effort="2.5"/>
         </joint>
         <link name="${prefix}_tibia">
@@ -170,16 +166,13 @@
         <joint name="${prefix}_elbow_joint" type="revolute">
             <xacro:if value="${left}">
-                <!-- <origin xyz="0.00 ${femur_thickness/2 - 0.0042} ${-femur_length}" rpy="0.0 ${-M_PI/2} 0.0"/> -->
-                <origin xyz="0.00 ${femur_thickness/2 - 0.0042} ${-femur_length}" rpy="0.0 0.0 0.0"/>
+                <origin xyz="0.00 ${femur_thickness/2 - 0.0042} ${-femur_length}" rpy="0.0 ${-M_PI/2} 0.0"/>
             </xacro:if>
             <xacro:unless value="${left}">
-                <!-- <origin xyz="0.00 ${-femur_thickness/2 + 0.0042} ${-femur_length}" rpy="0.0 ${-M_PI/2} 0.0"/> -->
-                <origin xyz="0.00 ${-femur_thickness/2 + 0.0042} ${-femur_length}" rpy="0.0 0.0 0.0"/>
+                <origin xyz="0.00 ${-femur_thickness/2 + 0.0042} ${-femur_length}" rpy="0.0 ${-M_PI/2} 0.0"/>
             </xacro:unless>
             <parent link="${prefix}_femur"/>
             <child link="${prefix}_tibia"/>
             <axis xyz="0 1 0"/>
-            <!-- <limit lower="${-M_PI/5}" upper="${M_PI/5}" velocity="5.75" effort="2.5"/> -->
-            <limit lower="${-M_PI}" upper="${M_PI}" velocity="5.75" effort="2.5"/>
+            <limit lower="${-M_PI/5}" upper="${M_PI/5}" velocity="5.75" effort="2.5"/>
         </joint>
         <link name="${prefix}_foot"/>

Commit message: Implement body IK transformation matrices

File: black_mouth_description/urdf/black_mouth.urdf.xacro (robot description, xacro)
@@ -12,5 +12,5 @@
     <xacro:property name="leg_x_offset" value="0.11455"/>
     <xacro:property name="leg_y_offset" value="0.07"/>
-    <xacro:property name="leg_z_offset" value="0.020822"/>
+    <xacro:property name="leg_z_offset" value="0.0208"/>
     <xacro:macro name="leg" params="prefix left front *joint_pose">
         <link name="${prefix}_hip_fixed">
@@ -186,4 +186,5 @@
     <link name="base_link">
         <visual>
+            <origin xyz="0.0 0.0 ${-leg_z_offset}" rpy="0.0 0.0 0.0"/>
             <geometry>
                 <mesh filename="file://$(find black_mouth_description)/meshes/base_link.dae" />
@@ -191,4 +192,5 @@
         </visual>
         <collision>
+            <origin xyz="0.0 0.0 ${-leg_z_offset}" rpy="0.0 0.0 0.0"/>
             <geometry>
                 <mesh filename="file://$(find black_mouth_description)/meshes/base_link.stl"/>
@@ -197,5 +199,5 @@
         <inertial>
             <mass value="1.28"/>
-            <origin xyz="0.0015 1.622e-4 0.0238" rpy="0.0 0.0 0.0"/>
+            <origin xyz="0.0015 1.622e-4 ${0.0238-leg_z_offset}" rpy="0.0 0.0 0.0"/>
             <inertia ixx="0.00327123" ixy="-2.696e-6" ixz="-1.456e-5" iyy="0.00459934" iyz="-1.166e-5" izz="0.00718769"/>
         </inertial>
@@ -214,17 +216,17 @@
         <parent link="base_footprint"/>
         <child link="base_link"/>
-        <origin xyz="0.0 0.0 0.15" rpy="0.0 0.0 0.0"/>
+        <origin xyz="0.0 0.0 0.17" rpy="0.0 0.0 0.0"/>
     </joint>
     <xacro:leg prefix="front_left" left="${True}" front="${True}">
-        <origin xyz="${leg_x_offset} ${leg_y_offset} ${leg_z_offset}" rpy="0.0 0.0 0.0"/>
+        <origin xyz="${leg_x_offset} ${leg_y_offset} 0.0" rpy="0.0 0.0 0.0"/>
     </xacro:leg>
     <xacro:leg prefix="front_right" left="${False}" front="${True}">
-        <origin xyz="${leg_x_offset} ${-leg_y_offset} ${leg_z_offset}" rpy="0.0 0.0 0.0"/>
+        <origin xyz="${leg_x_offset} ${-leg_y_offset} 0.0" rpy="0.0 0.0 0.0"/>
     </xacro:leg>
     <xacro:leg prefix="back_left" left="${True}" front="${False}">
-        <origin xyz="${-leg_x_offset} ${leg_y_offset} ${leg_z_offset}" rpy="0.0 0.0 0.0"/>
+        <origin xyz="${-leg_x_offset} ${leg_y_offset} 0.0" rpy="0.0 0.0 0.0"/>
     </xacro:leg>
     <xacro:leg prefix="back_right" left="${False}" front="${False}" >
-        <origin xyz="${-leg_x_offset} ${-leg_y_offset} ${leg_z_offset}" rpy="0.0 0.0 0.0"/>
+        <origin xyz="${-leg_x_offset} ${-leg_y_offset} 0.0" rpy="0.0 0.0 0.0"/>
     </xacro:leg>
     <link name="imu_link"/>

Commit message: Implement body IK transformation matrices

File: black_mouth_description/urdf/black_mouth.urdf.xacro (robot description, xacro)
@@ -12,5 +12,5 @@
     <xacro:property name="leg_x_offset" value="0.11455"/>
     <xacro:property name="leg_y_offset" value="0.07"/>
-    <xacro:property name="leg_z_offset" value="0.020822"/>
+    <xacro:property name="leg_z_offset" value="0.0208"/>
     <xacro:property name="effort_limit" value="0.01"/>
     <xacro:macro name="leg" params="prefix left front *joint_pose">
@@ -194,4 +194,5 @@
     <link name="base_link">
         <visual>
+            <origin xyz="0.0 0.0 ${-leg_z_offset}" rpy="0.0 0.0 0.0"/>
             <geometry>
                 <mesh filename="file://$(find black_mouth_description)/meshes/base_link.dae" />
@@ -199,4 +200,5 @@
         </visual>
         <collision>
+            <origin xyz="0.0 0.0 ${-leg_z_offset}" rpy="0.0 0.0 0.0"/>
             <geometry>
                 <mesh filename="file://$(find black_mouth_description)/meshes/base_link.stl"/>
@@ -205,5 +207,5 @@
         <inertial>
             <mass value="1.28"/>
-            <origin xyz="0.0015 1.622e-4 0.0238" rpy="0.0 0.0 0.0"/>
+            <origin xyz="0.0015 1.622e-4 ${0.0238-leg_z_offset}" rpy="0.0 0.0 0.0"/>
             <inertia ixx="0.00327123" ixy="-2.696e-6" ixz="-1.456e-5" iyy="0.00459934" iyz="-1.166e-5" izz="0.00718769"/>
         </inertial>
@@ -222,17 +224,17 @@
         <parent link="base_footprint"/>
         <child link="base_link"/>
-        <origin xyz="0.0 0.0 0.15" rpy="0.0 0.0 0.0"/>
+        <origin xyz="0.0 0.0 0.17" rpy="0.0 0.0 0.0"/>
     </joint>
     <xacro:leg prefix="front_left" left="${True}" front="${True}">
-        <origin xyz="${leg_x_offset} ${leg_y_offset} ${leg_z_offset}" rpy="0.0 0.0 0.0"/>
+        <origin xyz="${leg_x_offset} ${leg_y_offset} 0.0" rpy="0.0 0.0 0.0"/>
     </xacro:leg>
     <xacro:leg prefix="front_right" left="${False}" front="${True}">
-        <origin xyz="${leg_x_offset} ${-leg_y_offset} ${leg_z_offset}" rpy="0.0 0.0 0.0"/>
+        <origin xyz="${leg_x_offset} ${-leg_y_offset} 0.0" rpy="0.0 0.0 0.0"/>
     </xacro:leg>
     <xacro:leg prefix="back_left" left="${True}" front="${False}">
-        <origin xyz="${-leg_x_offset} ${leg_y_offset} ${leg_z_offset}" rpy="0.0 0.0 0.0"/>
-    </xacro:leg>
-    <xacro:leg prefix="back_right" left="${False}" front="${False}">
-        <origin xyz="${-leg_x_offset} ${-leg_y_offset} ${leg_z_offset}" rpy="0.0 0.0 0.0"/>
+        <origin xyz="${-leg_x_offset} ${leg_y_offset} 0.0" rpy="0.0 0.0 0.0"/>
+    </xacro:leg>
+    <xacro:leg prefix="back_right" left="${False}" front="${False}" >
+        <origin xyz="${-leg_x_offset} ${-leg_y_offset} 0.0" rpy="0.0 0.0 0.0"/>
     </xacro:leg>
     <link name="imu_link"/>

Commit message: test effort

File: black_mouth_description/urdf/black_mouth.urdf.xacro (robot description, xacro)
@@ -13,5 +13,5 @@
     <xacro:property name="leg_y_offset" value="0.07"/>
     <xacro:property name="leg_z_offset" value="0.020822"/>
-    <xacro:property name="effort_limit" value="0.01"/>
+    <xacro:property name="effort_limit" value="1"/>
     <xacro:macro name="leg" params="prefix left front *joint_pose">
         <link name="${prefix}_hip">

Commit message: setting pid values

File: black_mouth_description/urdf/black_mouth.urdf.xacro (robot description, xacro)
@@ -13,5 +13,5 @@
     <xacro:property name="leg_y_offset" value="0.07"/>
     <xacro:property name="leg_z_offset" value="0.020822"/>
-    <xacro:property name="effort_limit" value="1"/>
+    <xacro:property name="effort_limit" value="2"/>
     <xacro:macro name="leg" params="prefix left front *joint_pose">
         <link name="${prefix}_hip">
@@ -71,5 +71,5 @@
             <limit lower="${-M_PI/6}" upper="${M_PI/6}" velocity="5.75" effort="${effort_limit}"/>
             <xacro:insert_block name="joint_pose"/>
-            <!-- <dynamics damping="5.0" friction="5.0" /> -->
+            <dynamics damping="0.1" friction="0.01" />
         </joint>
         <link name="${prefix}_link_femur">
@@ -125,5 +125,5 @@
             <axis xyz="0 1 0"/>
             <limit lower="${-M_PI/4}" upper="${M_PI/4}" velocity="5.75" effort="${effort_limit}"/>
-            <!-- <dynamics damping="5.0" friction="5.0" /> -->
+            <dynamics damping="0.1" friction="0.01" />
         </joint>
         <link name="${prefix}_tibia">
@@ -165,5 +165,5 @@
             <axis xyz="0 1 0"/>
             <limit lower="${-M_PI/5}" upper="${M_PI/5}" velocity="5.75" effort="${effort_limit}"/>
-            <!-- <dynamics damping="5.0" friction="5.0" /> -->
+            <dynamics damping="0.00" friction="0.01" />
         </joint>
     </xacro:macro>

Commit message: fix merge

File: black_mouth_description/urdf/black_mouth.urdf.xacro (robot description, xacro)
@@ -14,5 +14,5 @@
     <xacro:property name="leg_z_offset" value="0.0208"/>
     <xacro:property name="effort_limit" value="2"/>
-    <xacro:macro name="leg" params="prefix left icont *joint_pose">
+    <xacro:macro name="leg" params="prefix left front *joint_pose">
         <link name="${prefix}_hip_fixed">
             <collision>

Commit message: Adjust yaw in real robot

File: black_mouth_description/urdf/black_mouth.urdf.xacro (robot description, xacro)
@@ -86,5 +86,5 @@
             <child link="${prefix}_hip"/>
             <axis xyz="1 0 0"/>
-            <limit lower="${-M_PI/6}" upper="${M_PI/6}" velocity="5.75" effort="${effort_limit}"/>
+            <limit lower="${-M_PI/4}" upper="${M_PI/4}" velocity="5.75" effort="${effort_limit}"/>
             <xacro:insert_block name="joint_pose"/>
             <dynamics damping="0.1" friction="0.01" />
@@ -141,5 +141,5 @@
             <child link="${prefix}_femur"/>
             <axis xyz="0 1 0"/>
-            <limit lower="${-M_PI/4}" upper="${M_PI/4}" velocity="5.75" effort="${effort_limit}"/>
+            <limit lower="${-M_PI/3}" upper="${M_PI/3}" velocity="5.75" effort="${effort_limit}"/>
             <dynamics damping="0.1" friction="0.01" />
         </joint>

File: black_mouth_description/urdf/black_mouth_real.urdf.xacro (robot description, xacro)
@@ -86,5 +86,5 @@
             <child link="${prefix}_hip"/>
             <axis xyz="1 0 0"/>
-            <limit lower="${-M_PI/6}" upper="${M_PI/6}" velocity="5.75" effort="${effort_limit}"/>
+            <limit lower="${-M_PI/4}" upper="${M_PI/4}" velocity="5.75" effort="${effort_limit}"/>
             <xacro:insert_block name="joint_pose"/>
             <dynamics damping="0.1" friction="0.01" />
@@ -141,5 +141,5 @@
             <child link="${prefix}_femur"/>
             <axis xyz="0 1 0"/>
-            <limit lower="${-M_PI/4}" upper="${M_PI/4}" velocity="5.75" effort="${effort_limit}"/>
+            <limit lower="${-M_PI/3}" upper="${M_PI/3}" velocity="5.75" effort="${effort_limit}"/>
             <dynamics damping="0.1" friction="0.01" />
         </joint>
