Commit message: urdf fixing

File: caramel_description/urdf/caramel.urdf.xacro (robot description, xacro)
@@ -201,5 +201,5 @@
             <origin xyz="0.0 0.0 ${-leg_z_offset}" rpy="0.0 0.0 0.0"/>
             <geometry>
-                <mesh filename="file://$(find caramel_description)/meshes/base_link.dae" />
+                <mesh filename="file://$(find caramel_description)/meshes/base.dae" />
             </geometry>
         </visual>
@@ -207,5 +207,5 @@
             <origin xyz="0.0 0.0 ${-leg_z_offset}" rpy="0.0 0.0 0.0"/>
             <geometry>
-                <mesh filename="file://$(find caramel_description)/meshes/base_link.stl"/>
+                <mesh filename="file://$(find caramel_description)/meshes/base_collision.stl"/>
             </geometry>
         </collision>

Commit message: xacro fix

File: caramel_description/urdf/caramel.urdf.xacro (robot description, xacro)
@@ -2,16 +2,16 @@
 <robot xmlns:xacro="http://www.ros.org/wiki/xacro" name="quadruped">
     <xacro:property name="M_PI" value="3.1415"/>
-    <xacro:property name="body_length" value="0.272"/>
-    <xacro:property name="body_width" value="0.168"/>
-    <xacro:property name="body_height" value="0.064"/>
+    <xacro:property name="body_length" value="0.290"/>
+    <xacro:property name="body_width" value="0.178"/>
+    <xacro:property name="body_height" value="0.063"/>
     <xacro:property name="L" value="0.2291"/>
     <xacro:property name="W" value="0.14"/>
     <xacro:property name="H" value="0.17"/>
     <xacro:property name="L1" value="0.048"/>
-    <xacro:property name="hip_length" value="0.0415"/>
-    <xacro:property name="femur_length" value="0.120"/>
-    <xacro:property name="tibia_length" value="0.120"/>
+    <xacro:property name="hip_length" value="0.045"/>
+    <xacro:property name="femur_length" value="0.126"/>
+    <xacro:property name="tibia_length" value="0.12"/>
     <xacro:property name="femur_thickness" value="0.022"/>
-    <xacro:property name="femur_offset" value="0.0053"/>
+    <xacro:property name="femur_offset" value="0.0"/>
     <xacro:property name="leg_x_offset" value="0.11455"/>
     <xacro:property name="leg_y_offset" value="0.07"/>
@@ -60,11 +60,11 @@
             <collision>
                 <xacro:if value="${front}">
-                    <origin xyz="-0.0149 0.0 0.0" rpy="0.0 0.0 0.0"/>
+                    <origin xyz="0.0 0.0 0.0" rpy="0.0 0.0 0.0"/>
                 </xacro:if>
                 <xacro:unless value="${front}">
-                    <origin xyz="0.0149 0.0 0.0" rpy="0.0 0.0 0.0"/>
-                </xacro:unless>
-                <geometry>
-                    <box size="0.0538 0.036 0.036"/>
+                    <origin xyz="0.0 0.0 0.0" rpy="0.0 0.0 0.0"/>
+                </xacro:unless>
+                <geometry>
+                    <box size="0.06 0.034 0.0385"/>
                 </geometry>
             </collision>
@@ -96,5 +96,5 @@
         <link name="${prefix}_femur">
             <visual>
-                <origin xyz="0.0 0 ${-femur_offset}" rpy="0.0 0.0 0.0 "/>
+                <origin xyz="0.0 0 ${-femur_offset}" rpy="0.0 0.0 0.0"/>
                 <geometry>
                     <xacro:if value="${left}">
@@ -111,5 +111,5 @@
                 </xacro:if>
                 <xacro:unless value="${left}">
-                    <origin xyz="0.0 0.0 ${-femur_offset}" rpy="0.0 0.0 ${M_PI}"/>
+                    <origin xyz="0.0 0.0 ${-femur_offset}" rpy="0.0 0.0 0.0"/>
                 </xacro:unless>
                 <geometry>
@@ -211,7 +211,7 @@
         </collision>
         <inertial>
-            <mass value="1.28"/>
-            <origin xyz="0.0015 1.622e-4 ${0.0238-leg_z_offset}" rpy="0.0 0.0 0.0"/>
-            <inertia ixx="0.00327123" ixy="-2.696e-6" ixz="-1.456e-5" iyy="0.00459934" iyz="-1.166e-5" izz="0.00718769"/>
+            <mass value="1.3"/>
+            <origin xyz="0.02 0 ${0.026-leg_z_offset}" rpy="0.0 0.0 0.0"/>
+            <inertia ixx="0.002671797" ixy="-1.86e-9" ixz="-5.8e-5" iyy="0.006415281" iyz="0" izz="0.008438753"/>
         </inertial>
     </link>

Commit message: fix urdf meshes and collisions

File: caramel_description/urdf/caramel.urdf.xacro (robot description, xacro)
@@ -17,5 +17,5 @@
     <xacro:property name="leg_y_offset" value="0.07"/>
     <xacro:property name="leg_z_offset" value="0.0208"/>
-    <xacro:property name="effort_limit" value="2"/>
+    <xacro:property name="effort_limit" value="20"/>
     <xacro:macro name="leg" params="prefix left front *joint_pose">
         <link name="${prefix}_hip_fixed">
@@ -111,5 +111,5 @@
                 </xacro:if>
                 <xacro:unless value="${left}">
-                    <origin xyz="0.0 0.0 ${-femur_offset}" rpy="0.0 0.0 0.0"/>
+                    <origin xyz="0.0 0.0 ${-femur_offset}" rpy="0.0 0.0 ${M_PI}"/>
                 </xacro:unless>
                 <geometry>

Commit message: fix urdf

File: caramel_description/urdf/caramel.urdf.xacro (robot description, xacro)
@@ -13,6 +13,6 @@
     <xacro:property name="tibia_length" value="0.12"/>
     <xacro:property name="femur_thickness" value="0.022"/>
-    <xacro:property name="femur_offset" value="0.0"/>
-    <xacro:property name="leg_x_offset" value="0.11455"/>
+    <xacro:property name="femur_offset" value="0.01"/>
+    <xacro:property name="leg_x_offset" value="0.125"/>
     <xacro:property name="leg_y_offset" value="0.07"/>
     <xacro:property name="leg_z_offset" value="0.0208"/>
@@ -60,8 +60,8 @@
             <collision>
                 <xacro:if value="${front}">
-                    <origin xyz="0.0 0.0 0.0" rpy="0.0 0.0 0.0"/>
+                    <origin xyz="-0.0152 0.0 0.0" rpy="0.0 0.0 0.0"/>
                 </xacro:if>
                 <xacro:unless value="${front}">
-                    <origin xyz="0.0 0.0 0.0" rpy="0.0 0.0 0.0"/>
+                    <origin xyz="0.0152 0.0 0.0" rpy="0.0 0.0 0.0"/>
                 </xacro:unless>
                 <geometry>
@@ -96,5 +96,5 @@
         <link name="${prefix}_femur">
             <visual>
-                <origin xyz="0.0 0 ${-femur_offset}" rpy="0.0 0.0 0.0"/>
+                <origin xyz="0.0 0 0.0" rpy="0.0 0.0 0.0"/>
                 <geometry>
                     <xacro:if value="${left}">
