Commit message: FIX HOPF PARAMS

File: caramel_control/urdf/real_robot.urdf.xacro (robot description, xacro)
@@ -4,9 +4,9 @@
         <hardware>
             <plugin>caramel_control/CaramelHW</plugin>
-            <param name="baud_rate">1000000</param>
+            <param name="baud_rate">4000000</param>
             <param name="usb_port">/dev/u2d2</param>
-            <param name="return_delay_type">100</param>
+            <param name="return_delay_type">0</param>
+            <param name="pd_control">false</param>
         </hardware>
-        <!-- FRONT RIGHT -->
         <joint name="front_right_hip_roll_joint">
             <param name="id">11</param>
@@ -15,7 +15,9 @@
             <param name="max_pos_limit">2386</param>
             <param name="home_angle">2048</param>
-            <param name="kp_gain">200</param>
-            <param name="ki_gain">450</param>
-            <param name="kd_gain">0</param>
+            <param name="kp_gain">300</param>
+            <param name="ki_gain">200</param>
+            <param name="kd_gain">0</param>
+            <param name="ctrl_kp">3.5</param>
+            <param name="ctrl_kd">0.02</param>
             <command_interface name="position">
                 <param name="min">-0.52</param>
@@ -30,7 +32,9 @@
             <param name="max_pos_limit">2048</param>
             <param name="home_angle">1533</param>
-            <param name="kp_gain">200</param>
-            <param name="ki_gain">450</param>
-            <param name="kd_gain">0</param>
+            <param name="kp_gain">300</param>
+            <param name="ki_gain">200</param>
+            <param name="kd_gain">0</param>
+            <param name="ctrl_kp">3.5</param>
+            <param name="ctrl_kd">0.02</param>
             <command_interface name="position">
                 <param name="min">-0.79</param>
@@ -45,14 +49,15 @@
             <param name="max_pos_limit">2490</param>
             <param name="home_angle">2048</param>
-            <param name="kp_gain">200</param>
-            <param name="ki_gain">450</param>
-            <param name="kd_gain">0</param>
-            <command_interface name="position">
-                <param name="min">-0.63</param>
-                <param name="max">0.63</param>
-            </command_interface>
-            <state_interface name="position"/>
-        </joint>
-        <!-- FRONT LEFT -->
+            <param name="kp_gain">300</param>
+            <param name="ki_gain">200</param>
+            <param name="kd_gain">0</param>
+            <param name="ctrl_kp">3.5</param>
+            <param name="ctrl_kd">0.02</param>
+            <command_interface name="position">
+                <param name="min">-0.63</param>
+                <param name="max">0.63</param>
+            </command_interface>
+            <state_interface name="position"/>
+        </joint>
         <joint name="front_left_hip_roll_joint">
             <param name="id">21</param>
@@ -61,7 +66,9 @@
             <param name="max_pos_limit">2386</param>
             <param name="home_angle">2048</param>
-            <param name="kp_gain">200</param>
-            <param name="ki_gain">450</param>
-            <param name="kd_gain">0</param>
+            <param name="kp_gain">300</param>
+            <param name="ki_gain">200</param>
+            <param name="kd_gain">0</param>
+            <param name="ctrl_kp">3.5</param>
+            <param name="ctrl_kd">0.02</param>
             <command_interface name="position">
                 <param name="min">-0.52</param>
@@ -76,7 +83,9 @@
             <param name="max_pos_limit">2048</param>
             <param name="home_angle">1533</param>
-            <param name="kp_gain">200</param>
-            <param name="ki_gain">450</param>
-            <param name="kd_gain">0</param>
+            <param name="kp_gain">300</param>
+            <param name="ki_gain">200</param>
+            <param name="kd_gain">0</param>
+            <param name="ctrl_kp">3.5</param>
+            <param name="ctrl_kd">0.02</param>
             <command_interface name="position">
                 <param name="min">-0.79</param>
@@ -91,14 +100,15 @@
             <param name="max_pos_limit">2490</param>
             <param name="home_angle">2048</param>
-            <param name="kp_gain">200</param>
-            <param name="ki_gain">450</param>
-            <param name="kd_gain">0</param>
-            <command_interface name="position">
-                <param name="min">-0.63</param>
-                <param name="max">0.63</param>
-            </command_interface>
-            <state_interface name="position"/>
-        </joint>
-        <!-- BACK RIGHT -->
+            <param name="kp_gain">300</param>
+            <param name="ki_gain">200</param>
+            <param name="kd_gain">0</param>
+            <param name="ctrl_kp">3.5</param>
+            <param name="ctrl_kd">0.02</param>
+            <command_interface name="position">
+                <param name="min">-0.63</param>
+                <param name="max">0.63</param>
+            </command_interface>
+            <state_interface name="position"/>
+        </joint>
         <joint name="back_right_hip_roll_joint">
             <param name="id">41</param>
@@ -107,7 +117,9 @@
             <param name="max_pos_limit">2386</param>
             <param name="home_angle">2048</param>
-            <param name="kp_gain">200</param>
-            <param name="ki_gain">450</param>
-            <param name="kd_gain">0</param>
+            <param name="kp_gain">300</param>
+            <param name="ki_gain">200</param>
+            <param name="kd_gain">0</param>
+            <param name="ctrl_kp">3.5</param>
+            <param name="ctrl_kd">0.02</param>
             <command_interface name="position">
                 <param name="min">-0.52</param>
@@ -122,7 +134,9 @@
             <param name="max_pos_limit">2048</param>
             <param name="home_angle">1533</param>
-            <param name="kp_gain">200</param>
-            <param name="ki_gain">450</param>
-            <param name="kd_gain">0</param>
+            <param name="kp_gain">300</param>
+            <param name="ki_gain">200</param>
+            <param name="kd_gain">0</param>
+            <param name="ctrl_kp">3.5</param>
+            <param name="ctrl_kd">0.02</param>
             <command_interface name="position">
                 <param name="min">-0.79</param>
@@ -137,14 +151,15 @@
             <param name="max_pos_limit">2490</param>
             <param name="home_angle">2048</param>
-            <param name="kp_gain">200</param>
-            <param name="ki_gain">450</param>
-            <param name="kd_gain">0</param>
-            <command_interface name="position">
-                <param name="min">-0.63</param>
-                <param name="max">0.63</param>
-            </command_interface>
-            <state_interface name="position"/>
-        </joint>
-        <!-- BACK LEFT -->
+            <param name="kp_gain">300</param>
+            <param name="ki_gain">200</param>
+            <param name="kd_gain">0</param>
+            <param name="ctrl_kp">3.5</param>
+            <param name="ctrl_kd">0.02</param>
+            <command_interface name="position">
+                <param name="min">-0.63</param>
+                <param name="max">0.63</param>
+            </command_interface>
+            <state_interface name="position"/>
+        </joint>
         <joint name="back_left_hip_roll_joint">
             <param name="id">31</param>
@@ -153,7 +168,9 @@
             <param name="max_pos_limit">2386</param>
             <param name="home_angle">2048</param>
-            <param name="kp_gain">200</param>
-            <param name="ki_gain">450</param>
-            <param name="kd_gain">0</param>
+            <param name="kp_gain">300</param>
+            <param name="ki_gain">200</param>
+            <param name="kd_gain">0</param>
+            <param name="ctrl_kp">3.5</param>
+            <param name="ctrl_kd">0.02</param>
             <command_interface name="position">
                 <param name="min">-0.52</param>
@@ -168,7 +185,9 @@
             <param name="max_pos_limit">2048</param>
             <param name="home_angle">1533</param>
-            <param name="kp_gain">200</param>
-            <param name="ki_gain">450</param>
-            <param name="kd_gain">0</param>
+            <param name="kp_gain">300</param>
+            <param name="ki_gain">200</param>
+            <param name="kd_gain">0</param>
+            <param name="ctrl_kp">3.5</param>
+            <param name="ctrl_kd">0.02</param>
             <command_interface name="position">
                 <param name="min">-0.79</param>
@@ -183,7 +202,9 @@
             <param name="max_pos_limit">2490</param>
             <param name="home_angle">2048</param>
-            <param name="kp_gain">200</param>
-            <param name="ki_gain">450</param>
-            <param name="kd_gain">0</param>
+            <param name="kp_gain">300</param>
+            <param name="ki_gain">200</param>
+            <param name="kd_gain">0</param>
+            <param name="ctrl_kp">3.5</param>
+            <param name="ctrl_kd">0.02</param>
             <command_interface name="position">
                 <param name="min">-0.63</param>
